File: TheMill.kicad_pcb (KiCad board)
At the start: 2 copper layers, 191.8 x 77.5 mm, 30 parts, among them U1 74LS32, U10 74LS245, U11 2716, U12 74LS367, U13 74LS367, U14 74LS367, U2 74LS08, U3 74LS266, U4 74LS74, U5 74LS30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

Commit message: 20190101 pcb ordered
Parts:
- removed C4: C, Apple2_bus:C_Disc_D4.3mm_W1.9mm_P5.00mm
- R1: value 470 -> 2.2k
- R2: value 10k -> 470
Routing:
- net Net-(U14-Pad6): track 153.2 -> 133.2 mm
- net +5V: track 541.1 -> 527.3 mm, vias 6 -> 5
- net Net-(U1-Pad3): track 132.3 -> 145.9 mm
- net GND: track 631.7 -> 622.1 mm, vias 12 -> 11
- net Net-(BUS1-Pad30): track 223.8 -> 217.2 mm
- net Net-(U13-Pad12): track 129.3 -> 134.3 mm
- net Net-(BUS1-Pad40): track 12.1 -> 16.4 mm
- net Net-(U3-Pad5): track 99.9 -> 96.8 mm
- net /a2: track 194.0 -> 196.7 mm
- net /a8: track 119.9 -> 117.8 mm
- net /a15: track 246.3 -> 244.5 mm
- net Net-(U3-Pad6): track 91.0 -> 92.8 mm
- net Net-(U12-Pad12): track 202.6 -> 201.0 mm
- net /da4: track 63.5 -> 62.0 mm
- net Net-(U7-Pad3): track 72.4 -> 70.9 mm
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- added copper zone on B.Cu, net Net-(U12-Pad1)
- removed copper zone on B.Cu, net GND
Other:
- net class Default: clearance 0.3048 -> 0.254; trace_width 0.2032 -> 0.381; via_dia 0.65 -> 1.016; via_drill 0.4 -> 0.508
- net class Power: clearance 0.3048 -> 0.254; trace_width 0.508 -> 1.27; via_dia 0.65 -> 1.016; via_drill 0.4 -> 0.508
- rule pad_to_mask_clearance: 0.2 -> 0.1778
- rule trace_clearance: 0.3048 -> 0.254
- rule trace_min: 0.2 -> 0.254
- rule via_min_drill: 0.3 -> 0.381
- rule via_min_size: 0.5 -> 0.762
- board text added: "The MILL Rev.A 1980 Original Design by James A. Hinds 2019 Remake by USHIRODA Atsushi"
- board text added: "nanja.info"
- board text removed: "The MILL"
