File: TheMill.sch (KiCad schematic (older format))
At the start: 30 parts, among them U1 74LS32, U10 74LS245, U11 2716, U12 74LS367, U13 74LS367, U14 74LS367, U2 74LS08, U3 74LS266, U4 74LS74, U5 74LS30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

Commit message: 20190101 pcb ordered
Parts:
- R1: value 470 -> 2.2k
- R2: value 10k -> 470
Changed lines of the file:
@@
 P 7050 4350
 F 0 "R1" V 6843 4350 50  0000 C CNN
-F 1 "470" V 6934 4350 50  0000 C CNN
+F 1 "2.2k" V 6934 4350 50  0000 C CNN
 F 2 "Apple2_bus:R_Axial_DIN0207_L6.3mm_D2.5mm_P10.16mm_Horizontal" V 6980 4350 50  0001 C CNN
 F 3 "~" H 7050 4350 50  0001 C CNN
@@
 P 3900 7850
 F 0 "R2" H 3970 7896 50  0000 L CNN
-F 1 "10k" H 3970 7805 50  0000 L CNN
+F 1 "470" H 3970 7805 50  0000 L CNN
 F 2 "Apple2_bus:R_Axial_DIN0207_L6.3mm_D2.5mm_P10.16mm_Horizontal" V 3830 7850 50  0001 C CNN
 F 3 "~" H 3900 7850 50  0001 C CNN
